Commit message: migrate from dlr git
Update xacro files (not completely) with parameters for effort and velocity and fixate the gripper (palm) to the world link.

File: robotiq_3f_gripper_visualization/cfg/fixed_robotiq-3f-gripper_articulated.xacro (robot description, xacro)
@@ -1,12 +1,4 @@
 <?xml version="1.0" ?>
 <robot name="robotiq-3f-gripper_articulated" xmlns:xacro="http://ros.org/wiki/xacro">
-    <!-- Add world and fixate the gripper with a joint -->
-    <link name="world"/>
-    <!--
-    <joint name="world_link" type="fixed">
-        <parent link="world"/>
-        <child link="tool00"/>
-        <origin xyz="0.0 0.0 0.0" rpy="0.0 0.0 0.0"/>
-    </joint> -->
     <!-- Insert 3f gripper -->
     <xacro:include filename="$(find robotiq_3f_gripper_visualization)/cfg/robotiq-3f-gripper_articulated_macro_transmissions.xacro" />
@@ -14,4 +6,11 @@
         <origin rpy="0 0 0" xyz="0 0 0"/>
     </xacro:robotiq-3f-gripper_articulated>
+    <!-- Load the Gazebo standard parameter "world" and fix the palm of the 3f-Gripper. -->
+    <link name="world"/>
+    <joint name="world_link" type="fixed">
+        <parent link="world"/>
+        <child link="palm"/>
+        <origin xyz="0.0 0.0 0.0" rpy="0.0 0.0 0.0"/>
+    </joint>
     <!--
       Inject Gazebo ROS Control plugin, which allows us to use ros_control

File: robotiq_3f_gripper_visualization/cfg/robotiq-3f-gripper_articulated_macro_transmissions.xacro (robot description, xacro)
@@ -1,5 +1,5 @@
 <robot xmlns:xacro="http://ros.org/wiki/xacro">
-        <xacro:property name="s1" value="0.85" />
-        <xacro:property name="e1" value="40" />
+        <xacro:property name="vel" value="1" />
+        <xacro:property name="eff" value="10" />
         <xacro:include filename="$(find robotiq_3f_gripper_visualization)/cfg/robotiq-3f-gripper_finger_articulated_macro.xacro" />
         <xacro:macro name="robotiq-3f-gripper_articulated" params="prefix *origin parent">
@@ -42,5 +42,5 @@
 			<axis xyz="0 1 0"/>
 			<origin xyz="-0.0455 0.0214 0.036" rpy="0 3.1416 -1.57"/>
-                        <limit lower="-0.1784" upper="0.192" effort="100" velocity="${s1}"/>
+                        <limit lower="-0.1784" upper="0.192" effort="${eff}" velocity="${vel}"/>
 		</joint>
 		<joint name="${prefix}palm_finger_2_joint" type="revolute">
@@ -49,5 +49,5 @@
 			<axis xyz="0 1 0"/>
 			<origin xyz="-0.0455 0.0214 -0.036" rpy="0 3.1416 -1.57"/>
-                        <limit lower="-0.192" upper="0.1784" effort="100" velocity="${s1}"/>
+                        <limit lower="-0.192" upper="0.1784" effort="${eff}" velocity="${vel}"/>
 		</joint>
 		<joint name="${prefix}palm_finger_middle_joint" type="fixed">
@@ -166,43 +166,4 @@
       </actuator>
     </transmission>
-	<!-- Configure self collision properties per link -->
-<!--  TODO: When active, model begins oscillating
-    <gazebo reference="${prefix}palm">
-      <selfCollide>true</selfCollide>
-    </gazebo>
-    <gazebo reference="${prefix}finger_1_link_0">
-      <selfCollide>true</selfCollide>
-    </gazebo>
-    <gazebo reference="${prefix}finger_1_link_1">
-      <selfCollide>true</selfCollide>
-    </gazebo>
-    <gazebo reference="${prefix}finger_1_link_2">
-      <selfCollide>true</selfCollide>
-    </gazebo>
-    <gazebo reference="${prefix}finger_1_link_3">
-      <selfCollide>true</selfCollide>
-    </gazebo>
-    <gazebo reference="${prefix}finger_2_link_0">
-      <selfCollide>true</selfCollide>
-    </gazebo>
-    <gazebo reference="${prefix}finger_2_link_1">
-      <selfCollide>true</selfCollide>
-    </gazebo>
-    <gazebo reference="${prefix}finger_2_link_2">
-      <selfCollide>true</selfCollide>
-    </gazebo>
-    <gazebo reference="${prefix}finger_2_link_3">
-      <selfCollide>true</selfCollide>
-    </gazebo>
-    <gazebo reference="${prefix}finger_middle_link_1">
-      <selfCollide>true</selfCollide>
-    </gazebo>
-    <gazebo reference="${prefix}finger_middle_link_2">
-      <selfCollide>true</selfCollide>
-    </gazebo>
-    <gazebo reference="${prefix}finger_middle_link_3">
-      <selfCollide>true</selfCollide>
-    </gazebo>
--->
 	</xacro:macro>
 </robot>

File: robotiq_3f_gripper_visualization/cfg/robotiq-3f-gripper_finger_articulated_macro.xacro (robot description, xacro)
@@ -1,9 +1,10 @@
 <!--
-robotiq-3f-gripper_finder_articulated_macro(prefix)
-Creates an articulated robotiq-3f-gripper finder with the passed in prefix.  The
+Creates an articulated Robotiq 3f-Gripper finder with the passed in prefix. The
 prefix typcially includes the hand prefix and an identifier for the
 finger(i.e. finger_1, etc...).
 -->
 <robot xmlns:xacro="http://ros.org/wiki/xacro">
+		<xacro:property name="vel" value="1" />
+    	<xacro:property name="eff" value="10" />
         <xacro:macro name="robotiq-3f-gripper_finger_articulated" params="prefix">
 		<!-- link list -->
@@ -108,5 +109,6 @@
 			<axis xyz="0 0 1"/>
 			<origin xyz="0.020 0 0" rpy="0 0 0"/>
-			<limit lower="0.0495" upper="1.2218" effort="100" velocity="100"/>
+			<limit lower="0.0495" upper="1.2218" effort="${eff}" velocity="${vel}"/>
+			<dynamics damping="0" friction="0"/>
 		</joint>
 		<joint name="${prefix}joint_2" type="revolute">
@@ -115,5 +117,6 @@
 			<axis xyz="0 0 1"/>
 			<origin xyz="0.050 -.028 0" rpy="0 0 -0.52"/>
-			<limit lower="0.0" upper="1.5708" effort="100" velocity="100"/>
+			<limit lower="0.0" upper="1.5708" effort="${eff}" velocity="${vel}"/>
+			<dynamics damping="0" friction="0"/>
 		</joint>
 		<joint name="${prefix}joint_3" type="revolute">
@@ -122,5 +125,6 @@
 			<axis xyz="0 0 1"/>
 			<origin xyz="0.039 0 0" rpy="0 0 0"/>
-			<limit lower="-1.2217" upper="-0.0523" effort="100" velocity="100"/>
+			<limit lower="-1.2217" upper="-0.0523" effort="${eff}" velocity="${vel}"/>
+			<dynamics damping="0" friction="0"/>
 		</joint>
 		<!-- end of joint list -->

Commit message: bugfix double call for joint between palm and world

File: robotiq_3f_gripper_visualization/cfg/fixed_robotiq-3f-gripper_articulated.xacro (robot description, xacro)
@@ -1,4 +1,6 @@
 <?xml version="1.0" ?>
 <robot name="robotiq-3f-gripper_articulated" xmlns:xacro="http://ros.org/wiki/xacro">
+    <!-- Load the Gazebo standard parameter "world" and fix the palm of the 3f-Gripper. -->
+    <link name="world"/>
     <!-- Insert 3f gripper -->
     <xacro:include filename="$(find robotiq_3f_gripper_visualization)/cfg/robotiq-3f-gripper_articulated_macro_transmissions.xacro" />
@@ -6,11 +8,4 @@
         <origin rpy="0 0 0" xyz="0 0 0"/>
     </xacro:robotiq-3f-gripper_articulated>
-    <!-- Load the Gazebo standard parameter "world" and fix the palm of the 3f-Gripper. -->
-    <link name="world"/>
-    <joint name="world_link" type="fixed">
-        <parent link="world"/>
-        <child link="palm"/>
-        <origin xyz="0.0 0.0 0.0" rpy="0.0 0.0 0.0"/>
-    </joint>
     <!--
       Inject Gazebo ROS Control plugin, which allows us to use ros_control
