Commit message: move .stl- and .dae-files and their path in xacro to convenient directory

File: robotiq_3f_gripper_visualization/cfg/robotiq-3f-gripper_articulated_macro.xacro (robot description, xacro)
@@ -10,5 +10,5 @@
 			<visual>
 				<geometry>
-                                        <mesh filename="package://robotiq_3f_gripper_visualization/meshes/robotiq-3f-gripper_articulated/visual/palm.dae" />
+                                        <mesh filename="package://robotiq_3f_gripper_visualization/meshes/visual/palm.dae" />
 				</geometry>
 				<material name="gray">
@@ -18,5 +18,5 @@
 			<collision>
 				<geometry>
-                                        <mesh filename="package://robotiq_3f_gripper_visualization/meshes/robotiq-3f-gripper_articulated/collision/palm.STL" />
+                                        <mesh filename="package://robotiq_3f_gripper_visualization/meshes/collision/palm.STL" />
 				</geometry>
 				<material name="yellow">

File: robotiq_3f_gripper_visualization/cfg/robotiq-3f-gripper_articulated_macro_transmissions.xacro (robot description, xacro)
@@ -11,5 +11,5 @@
 			<visual>
 				<geometry>
-                                        <mesh filename="package://robotiq_3f_gripper_visualization/meshes/robotiq-3f-gripper_articulated/visual/palm.dae" />
+                                        <mesh filename="package://robotiq_3f_gripper_visualization/meshes/visual/palm.dae" />
 				</geometry>
 				<material name="gray">
@@ -19,5 +19,5 @@
 			<collision>
 				<geometry>
-                                        <mesh filename="package://robotiq_3f_gripper_visualization/meshes/robotiq-3f-gripper_articulated/collision/palm.STL" />
+                                        <mesh filename="package://robotiq_3f_gripper_visualization/meshes/collision/palm.STL" />
 				</geometry>
 				<material name="yellow">

File: robotiq_3f_gripper_visualization/cfg/robotiq-3f-gripper_finger_articulated_macro.xacro (robot description, xacro)
@@ -13,5 +13,5 @@
 				<origin xyz="0.020 0 0" rpy="0 0 0"/>
 				<geometry>
-                                        <mesh filename="package://robotiq_3f_gripper_visualization/meshes/robotiq-3f-gripper_articulated/visual/link_0.dae" />
+                                        <mesh filename="package://robotiq_3f_gripper_visualization/meshes/visual/link_0.dae" />
 				</geometry>
 				<material name="gray">
@@ -22,5 +22,5 @@
 				<origin xyz="0.020 0 0" rpy="0 0 0"/>
 				<geometry>
-                                        <mesh filename="package://robotiq_3f_gripper_visualization/meshes/robotiq-3f-gripper_articulated/collision/link_0.STL" />
+                                        <mesh filename="package://robotiq_3f_gripper_visualization/meshes/collision/link_0.STL" />
 				</geometry>
 				<material name="yellow">
@@ -38,5 +38,5 @@
 				<origin xyz="0.050 -.028 0" rpy="0 0 -0.52"/>
 				<geometry>
-                                        <mesh filename="package://robotiq_3f_gripper_visualization/meshes/robotiq-3f-gripper_articulated/visual/link_1.dae" />
+                                        <mesh filename="package://robotiq_3f_gripper_visualization/meshes/visual/link_1.dae" />
 				</geometry>
 				<material name="gray"/>
@@ -45,5 +45,5 @@
 				<origin xyz="0.050 -.028 0" rpy="0 0 -0.52"/>
 				<geometry>
-                                        <mesh filename="package://robotiq_3f_gripper_visualization/meshes/robotiq-3f-gripper_articulated/collision/link_1.STL" />
+                                        <mesh filename="package://robotiq_3f_gripper_visualization/meshes/collision/link_1.STL" />
 				</geometry>
 				<material name="yellow"/>
@@ -64,5 +64,5 @@
 				<origin xyz="0.039 0 0.0075" rpy="0 0 0"/>
 				<geometry>
-                                        <mesh filename="package://robotiq_3f_gripper_visualization/meshes/robotiq-3f-gripper_articulated/visual/link_2.dae" />
+                                        <mesh filename="package://robotiq_3f_gripper_visualization/meshes/visual/link_2.dae" />
 				</geometry>
 				<material name="gray"/>
@@ -71,5 +71,5 @@
 				<origin xyz="0.039 0 0.0075" rpy="0 0 0"/>
 				<geometry>
-                                        <mesh filename="package://robotiq_3f_gripper_visualization/meshes/robotiq-3f-gripper_articulated/collision/link_2.STL" />
+                                        <mesh filename="package://robotiq_3f_gripper_visualization/meshes/collision/link_2.STL" />
 				</geometry>
 				<material name="yellow"/>
@@ -85,5 +85,5 @@
 				<origin xyz="0 0 0" rpy="0 0 0.52"/>
 				<geometry>
-                                        <mesh filename="package://robotiq_3f_gripper_visualization/meshes/robotiq-3f-gripper_articulated/visual/link_3.dae" />
+                                        <mesh filename="package://robotiq_3f_gripper_visualization/meshes/visual/link_3.dae" />
 				</geometry>
 				<material name="gray"/>
@@ -92,5 +92,5 @@
 				<origin xyz="0 0 0" rpy="0 0 0.52"/>
 				<geometry>
-                                        <mesh filename="package://robotiq_3f_gripper_visualization/meshes/robotiq-3f-gripper_articulated/collision/link_3.STL" />
+                                        <mesh filename="package://robotiq_3f_gripper_visualization/meshes/collision/link_3.STL" />
 				</geometry>
 				<material name="yellow"/>

File: robotiq_3f_gripper_visualization/cfg/robotiq_hand_macro.urdf.xacro (robot description, xacro)
@@ -14,5 +14,5 @@
         <origin xyz="0 0 0" rpy="0 0 0"/>
         <geometry>
-          <mesh filename="package://robotiq_3f_gripper_visualization/meshes/robotiq-3f-gripper_articulated/visual/link_0.dae" />
+          <mesh filename="package://robotiq_3f_gripper_visualization/meshes/visual/link_0.dae" />
         </geometry>
         <material name="green">
@@ -23,5 +23,5 @@
         <origin rpy="0 0 0" xyz="0 0 0"/>
         <geometry>
-          <mesh filename="package://robotiq_3f_gripper_visualization/meshes/robotiq-3f-gripper_articulated/collision/link_0.STL" />
+          <mesh filename="package://robotiq_3f_gripper_visualization/meshes/collision/link_0.STL" />
         </geometry>
         <material name="yellow">
@@ -44,5 +44,5 @@
         <origin rpy="0 0 ${3.1416/2}" xyz="0 0.05717 0"/>
         <geometry>
-          <mesh filename="package://robotiq_3f_gripper_visualization/meshes/robotiq-3f-gripper_articulated/visual/link_1.dae" />
+          <mesh filename="package://robotiq_3f_gripper_visualization/meshes/visual/link_1.dae" />
         </geometry>
         <material name="green"/>
@@ -51,5 +51,5 @@
         <origin rpy="0 0 ${3.1416/2}" xyz="0 0.05717 0"/>
         <geometry>
-          <mesh filename="package://robotiq_3f_gripper_visualization/meshes/robotiq-3f-gripper_articulated/collision/link_1.STL"/>
+          <mesh filename="package://robotiq_3f_gripper_visualization/meshes/collision/link_1.STL"/>
         </geometry>
         <material name="yellow">
@@ -77,5 +77,5 @@
         <origin rpy="0 0 ${3.1416/2}" xyz="0 0.03810 0.0075"/>
         <geometry>
-          <mesh filename="package://robotiq_3f_gripper_visualization/meshes/robotiq-3f-gripper_articulated/visual/link_2.dae" />
+          <mesh filename="package://robotiq_3f_gripper_visualization/meshes/visual/link_2.dae" />
         </geometry>
         <material name="green"/>
@@ -84,5 +84,5 @@
         <origin rpy="0 0 ${3.1416/2}" xyz="0 0.03810 0.0075"/>
           <geometry>
-            <mesh filename="package://robotiq_3f_gripper_visualization/meshes/robotiq-3f-gripper_articulated/collision/link_2.STL"/>
+            <mesh filename="package://robotiq_3f_gripper_visualization/meshes/collision/link_2.STL"/>
           </geometry>
         <material name="yellow"/>
@@ -108,5 +108,5 @@
         <origin xyz="0 0 0" rpy="0 0 0"/>
         <geometry>
-          <mesh filename="package://robotiq_3f_gripper_visualization/meshes/robotiq-3f-gripper_articulated/visual/link_3.dae" />
+          <mesh filename="package://robotiq_3f_gripper_visualization/meshes/visual/link_3.dae" />
         </geometry>
         <material name="green"/>
@@ -115,5 +115,5 @@
         <origin xyz="0 0 0" rpy="0 0 0"/>
         <geometry>
-          <mesh filename="package://robotiq_3f_gripper_visualization/meshes/robotiq-3f-gripper_articulated/collision/link_3.STL"/>
+          <mesh filename="package://robotiq_3f_gripper_visualization/meshes/collision/link_3.STL"/>
         </geometry>
         <material name="yellow"/>
@@ -648,5 +648,5 @@
         <visual>
           <geometry>
-            <mesh filename="package://robotiq_3f_gripper_visualization/meshes/robotiq-3f-gripper_articulated/visual/palm.dae" />
+            <mesh filename="package://robotiq_3f_gripper_visualization/meshes/visual/palm.dae" />
           </geometry>
           <material name="green">
