Commit message: adapt old macros with new parameters

File: robotiq_3f_description/urdf/inc/transmission_macro.xacro (robot description, xacro)
@@ -1,71 +1,10 @@
+<?xml version="1.0"?>
 <robot xmlns:xacro="http://ros.org/wiki/xacro">
-        <xacro:property name="vel" value="1" />
-        <xacro:property name="eff" value="10" />
-        <xacro:include filename="$(find robotiq_3f_gripper_visualization)/cfg/robotiq-3f-gripper_finger_articulated_macro.xacro" />
-        <xacro:macro name="robotiq-3f-gripper_articulated" params="prefix *origin parent">
-        <xacro:robotiq-3f-gripper_finger_articulated prefix="${prefix}finger_1_"/>
-        <xacro:robotiq-3f-gripper_finger_articulated prefix="${prefix}finger_2_"/>
-        <xacro:robotiq-3f-gripper_finger_articulated prefix="${prefix}finger_middle_"/>
-		<!-- link list -->
-		<link name="${prefix}palm">
-			<visual>
-				<geometry>
-                                        <mesh filename="package://robotiq_3f_gripper_visualization/meshes/visual/palm.dae" />
-				</geometry>
-				<material name="gray">
-					<color rgba="0.2 0.2 0.2 1"/>
-				</material>
-			</visual>
-			<collision>
-				<geometry>
-                                        <mesh filename="package://robotiq_3f_gripper_visualization/meshes/collision/palm.STL" />
-				</geometry>
-				<material name="yellow">
-					<color rgba="0 1 1 1"/>
-				</material>
-			</collision>
-		</link>
-	    <gazebo reference="${prefix}palm">
-      		<mu1>1.1</mu1>
-      		<mu2>1.1</mu2>
-    	</gazebo>
-        <inertial>
-            <origin xyz="0 0 0" rpy="0 0 0"/>
-            <mass value="1.3"/>
-            <inertia ixx="0.006012" ixy="0.000079" ixz="-0.00024" iyy="0.012892" iyz="0" izz="0.002435" />
-        </inertial>
-		<!-- end of link list -->
-		<!-- joint list -->
-		<joint name="${prefix}palm_finger_1_joint" type="revolute">
-			<parent link="${prefix}palm"/>
-			<child link="${prefix}finger_1_link_0"/>
-			<axis xyz="0 1 0"/>
-			<origin xyz="-0.0455 0.0214 0.036" rpy="0 3.1416 -1.57"/>
-                        <limit lower="-0.1784" upper="0.192" effort="${eff}" velocity="${vel}"/>
-		</joint>
-		<joint name="${prefix}palm_finger_2_joint" type="revolute">
-			<parent link="${prefix}palm"/>
-			<child link="${prefix}finger_2_link_0"/>
-			<axis xyz="0 1 0"/>
-			<origin xyz="-0.0455 0.0214 -0.036" rpy="0 3.1416 -1.57"/>
-                        <limit lower="-0.192" upper="0.1784" effort="${eff}" velocity="${vel}"/>
-		</joint>
-		<joint name="${prefix}palm_finger_middle_joint" type="fixed">
-			<parent link="${prefix}palm"/>
-			<child link="${prefix}finger_middle_link_0"/>
-			<axis xyz="0 0 1"/>
-			<origin xyz="0.0455 0.0214 0" rpy="0 0 1.57"/>
-		</joint>
-		<joint name="${prefix}robotiq_hand_joint" type="fixed">
-      		<xacro:insert_block name="origin"/>
-      		<parent link="${parent}"/>
-      		<child link="${prefix}palm"/>
-    	</joint>
-        <!-- end of joint list -->
+  <xacro:macro name="transmission" params="prefix hw_interface">
 	<!-- Palm transmission macro -->
     <transmission name="${prefix}palm_finger_1_trans">
       <type>transmission_interface/SimpleTransmission</type>
       <joint name="${prefix}palm_finger_1_joint">
-        <hardwareInterface>hardware_interface/EffortJointInterface</hardwareInterface>
+        <hardwareInterface>${hw_interface}</hardwareInterface>
       </joint>
       <actuator name="${prefix}palm_finger_1_motor">
@@ -76,5 +15,5 @@
       <type>transmission_interface/SimpleTransmission</type>
       <joint name="${prefix}palm_finger_2_joint">
-        <hardwareInterface>hardware_interface/EffortJointInterface</hardwareInterface>
+        <hardwareInterface>${hw_interface}</hardwareInterface>
       </joint>
       <actuator name="${prefix}palm_finger_2_motor">
@@ -86,5 +25,5 @@
       <type>transmission_interface/SimpleTransmission</type>
       <joint name="${prefix}finger_1_joint_1">
-        <hardwareInterface>hardware_interface/EffortJointInterface</hardwareInterface>
+        <hardwareInterface>${hw_interface}</hardwareInterface>
       </joint>
       <actuator name="${prefix}finger_1_motor_1">
@@ -95,5 +34,5 @@
       <type>transmission_interface/SimpleTransmission</type>
       <joint name="${prefix}finger_1_joint_2">
-        <hardwareInterface>hardware_interface/EffortJointInterface</hardwareInterface>
+        <hardwareInterface>${hw_interface}</hardwareInterface>
       </joint>
       <actuator name="${prefix}finger_1_motor_2">
@@ -104,5 +43,5 @@
       <type>transmission_interface/SimpleTransmission</type>
       <joint name="${prefix}finger_1_joint_3">
-        <hardwareInterface>hardware_interface/EffortJointInterface</hardwareInterface>
+        <hardwareInterface>${hw_interface}</hardwareInterface>
       </joint>
       <actuator name="${prefix}finger_1_motor_3">
@@ -114,5 +53,5 @@
       <type>transmission_interface/SimpleTransmission</type>
       <joint name="${prefix}finger_2_joint_1">
-        <hardwareInterface>hardware_interface/EffortJointInterface</hardwareInterface>
+        <hardwareInterface>${hw_interface}</hardwareInterface>
       </joint>
       <actuator name="${prefix}finger_2_motor_1">
@@ -123,5 +62,5 @@
       <type>transmission_interface/SimpleTransmission</type>
       <joint name="${prefix}finger_2_joint_2">
-        <hardwareInterface>hardware_interface/EffortJointInterface</hardwareInterface>
+        <hardwareInterface>${hw_interface}</hardwareInterface>
       </joint>
       <actuator name="${prefix}finger_2_motor_2">
@@ -132,5 +71,5 @@
       <type>transmission_interface/SimpleTransmission</type>
       <joint name="${prefix}finger_2_joint_3">
-        <hardwareInterface>hardware_interface/EffortJointInterface</hardwareInterface>
+        <hardwareInterface>${hw_interface}</hardwareInterface>
       </joint>
       <actuator name="${prefix}finger_2_motor_3">
@@ -142,5 +81,5 @@
       <type>transmission_interface/SimpleTransmission</type>
       <joint name="${prefix}finger_middle_joint_1">
-        <hardwareInterface>hardware_interface/EffortJointInterface</hardwareInterface>
+        <hardwareInterface>${hw_interface}</hardwareInterface>
       </joint>
       <actuator name="${prefix}finger_middle_motor_1">
@@ -151,5 +90,5 @@
       <type>transmission_interface/SimpleTransmission</type>
       <joint name="${prefix}finger_middle_joint_2">
-        <hardwareInterface>hardware_interface/EffortJointInterface</hardwareInterface>
+        <hardwareInterface>${hw_interface}</hardwareInterface>
       </joint>
       <actuator name="${prefix}finger_middle_motor_2">
@@ -160,5 +99,5 @@
       <type>transmission_interface/SimpleTransmission</type>
       <joint name="${prefix}finger_middle_joint_3">
-        <hardwareInterface>hardware_interface/EffortJointInterface</hardwareInterface>
+        <hardwareInterface>${hw_interface}</hardwareInterface>
       </joint>
       <actuator name="${prefix}finger_middle_motor_3">
@@ -166,4 +105,4 @@
       </actuator>
     </transmission>
-	</xacro:macro>
+  </xacro:macro>
 </robot>
