Commit message: move the static 3f transmission macro to a parameterized macro

File: robotiq_3f_description/urdf/inc/robotiq_common.xacro (robot description, xacro)
@@ -1,4 +1,20 @@
 <?xml version="1.0"?>
 <robot xmlns:xacro="http://wiki.ros.org/xacro">
+  <xacro:macro name="transmission" params="
+    joint_name
+    hw_interface
+    mechanical_reduction:=1"
+  >
+    <!-- Transmission macro -->
+    <transmission name="${joint_name}_trans">
+      <type>transmission_interface/SimpleTransmission</type>
+      <joint name="${joint_name}">
+        <hardwareInterface>${hw_interface}</hardwareInterface>
+      </joint>
+      <actuator name="${joint_name}_motor">
+        <mechanicalReduction>${mechanical_reduction}</mechanicalReduction>
+      </actuator>
+    </transmission>
+  </xacro:macro>
   <xacro:macro name="read_model_data" params="joint_limits_parameters_file physical_parameters_file visual_parameters_file">
     <!-- Read .yaml files from disk, load content into properties -->

File: robotiq_3f_description/urdf/robotiq_3f_macro.xacro (robot description, xacro)
@@ -3,5 +3,4 @@
   <xacro:include filename="inc/finger_macro.xacro"/>
   <xacro:include filename="inc/palm_macro.xacro"/>
-  <xacro:include filename="inc/transmission_macro.xacro"/>
   <xacro:include filename="inc/robotiq_common.xacro"/>
   <xacro:macro name="robotiq_3f_assembler" params="
@@ -37,5 +36,45 @@
     />
     <xacro:transmission
-      prefix="${prefix}"
+      joint_name="${prefix}palm_finger_1_joint"
+      hw_interface="${transmission_hw_interface}"
+    />
+    <xacro:transmission
+      joint_name="${prefix}palm_finger_2_joint"
+      hw_interface="${transmission_hw_interface}"
+    />
+    <xacro:transmission
+      joint_name="${prefix}finger_1_joint_1"
+      hw_interface="${transmission_hw_interface}"
+    />
+    <xacro:transmission
+      joint_name="${prefix}finger_1_joint_2"
+      hw_interface="${transmission_hw_interface}"
+    />
+    <xacro:transmission
+      joint_name="${prefix}finger_1_joint_3"
+      hw_interface="${transmission_hw_interface}"
+    />
+    <xacro:transmission
+      joint_name="${prefix}finger_2_joint_1"
+      hw_interface="${transmission_hw_interface}"
+    />
+    <xacro:transmission
+      joint_name="${prefix}finger_2_joint_2"
+      hw_interface="${transmission_hw_interface}"
+    />
+    <xacro:transmission
+      joint_name="${prefix}finger_2_joint_3"
+      hw_interface="${transmission_hw_interface}"
+    />
+    <xacro:transmission
+      joint_name="${prefix}finger_middle_joint_1"
+      hw_interface="${transmission_hw_interface}"
+    />
+    <xacro:transmission
+      joint_name="${prefix}finger_middle_joint_2"
+      hw_interface="${transmission_hw_interface}"
+    />
+    <xacro:transmission
+      joint_name="${prefix}finger_middle_joint_3"
       hw_interface="${transmission_hw_interface}"
     />
