Commit message: move origin parameters to parameter file (yaml)

File: robotiq_3f_description/urdf/inc/finger_macro.xacro (robot description, xacro)
@@ -20,5 +20,5 @@
     <link name="${prefix}link_0">
       <visual>
-        <origin xyz="0.020 0 0" rpy="0 0 0"/>
+        <origin xyz="${link_0_origin_xyz}" rpy="${link_0_origin_rpy}"/>
         <geometry>
           <mesh filename="${finger_link_0_visual_mesh}" />
@@ -29,5 +29,5 @@
       </visual>
       <collision>
-        <origin xyz="0.020 0 0" rpy="0 0 0"/>
+        <origin xyz="${link_0_origin_xyz}" rpy="${link_0_origin_rpy}"/>
         <geometry>
           <mesh filename="${finger_link_0_collision_mesh}" />
@@ -47,5 +47,5 @@
     <link name="${prefix}link_1">
       <visual>
-        <origin xyz="0.050 -.028 0" rpy="0 0 -0.52"/>
+        <origin xyz="${link_1_origin_xyz}" rpy="${link_1_origin_rpy}"/>
         <geometry>
           <mesh filename="${finger_link_1_visual_mesh}" />
@@ -56,5 +56,5 @@
       </visual>
       <collision>
-        <origin xyz="0.050 -.028 0" rpy="0 0 -0.52"/>
+        <origin xyz="${link_1_origin_xyz}" rpy="${link_1_origin_rpy}"/>
         <geometry>
           <mesh filename="${finger_link_1_collision_mesh}" />
@@ -79,5 +79,5 @@
       -->
       <visual>
-        <origin xyz="0.039 0 0.0075" rpy="0 0 0"/>
+        <origin xyz="${link_2_origin_xyz}" rpy="${link_2_origin_rpy}"/>
         <geometry>
           <mesh filename="${finger_link_2_visual_mesh}" />
@@ -88,5 +88,5 @@
       </visual>
       <collision>
-        <origin xyz="0.039 0 0.0075" rpy="0 0 0"/>
+        <origin xyz="${link_2_origin_xyz}" rpy="${link_2_origin_rpy}"/>
         <geometry>
           <mesh filename="${finger_link_2_collision_mesh}" />
@@ -106,5 +106,5 @@
     <link name="${prefix}link_3">
       <visual>
-        <origin xyz="0 0 0" rpy="0 0 0.52"/>
+        <origin xyz="${link_3_origin_xyz}" rpy="${link_3_origin_rpy}"/>
         <geometry>
           <mesh filename="${finger_link_3_visual_mesh}" />
@@ -115,5 +115,5 @@
       </visual>
       <collision>
-        <origin xyz="0 0 0" rpy="0 0 0.52"/>
+        <origin xyz="${link_3_origin_xyz}" rpy="${link_3_origin_rpy}"/>
         <geometry>
           <mesh filename="${finger_link_3_collision_mesh}" />
@@ -135,5 +135,5 @@
       <child link="${prefix}link_1"/>
       <axis xyz="0 0 1"/>
-      <origin xyz="0.020 0 0" rpy="0 0 0"/>
+      <origin xyz="${joint_1_origin_xyz}" rpy="${joint_1_origin_rpy}"/>
       <limit lower="${finger_joint_1_lower_limit}"
              upper="${finger_joint_1_upper_limit}"
@@ -146,5 +146,5 @@
       <child link="${prefix}link_2"/>
       <axis xyz="0 0 1"/>
-      <origin xyz="0.050 -.028 0" rpy="0 0 -0.52"/>
+      <origin xyz="${joint_2_origin_xyz}" rpy="${joint_2_origin_rpy}"/>
       <limit lower="${finger_joint_2_lower_limit}"
              upper="${finger_joint_2_upper_limit}"
@@ -157,5 +157,5 @@
       <child link="${prefix}link_3"/>
       <axis xyz="0 0 1"/>
-      <origin xyz="0.039 0 0" rpy="0 0 0"/>
+      <origin xyz="${joint_3_origin_xyz}" rpy="${joint_3_origin_rpy}"/>
       <limit lower="${finger_joint_3_lower_limit}"
              upper="${finger_joint_3_upper_limit}"

File: robotiq_3f_description/urdf/inc/palm_macro.xacro (robot description, xacro)
@@ -37,5 +37,5 @@
       <child link="${prefix}finger_1_link_0"/>
       <axis xyz="0 1 0"/>
-      <origin xyz="-0.0455 0.0214 0.036" rpy="0 3.1416 -1.57"/>
+      <origin xyz="${palm_finger_1_joint_origin_xyz}" rpy="${palm_finger_1_joint_origin_rpy}"/>
       <limit lower="${palm_finger_1_joint_lower_limit}"
              upper="${palm_finger_1_joint_upper_limit}"
@@ -47,5 +47,5 @@
       <child link="${prefix}finger_2_link_0"/>
       <axis xyz="0 1 0"/>
-      <origin xyz="-0.0455 0.0214 -0.036" rpy="0 3.1416 -1.57"/>
+      <origin xyz="${palm_finger_2_joint_origin_xyz}" rpy="${palm_finger_2_joint_origin_rpy}"/>
       <limit lower="${palm_finger_2_joint_lower_limit}"
              upper="${palm_finger_2_joint_upper_limit}"
@@ -57,5 +57,5 @@
       <child link="${prefix}finger_middle_link_0"/>
       <axis xyz="0 0 1"/>
-      <origin xyz="0.0455 0.0214 0" rpy="0 0 1.57"/>
+      <origin xyz="${palm_finger_middle_joint_origin_xyz}" rpy="${palm_finger_middle_joint_origin_rpy}"/>
     </joint>
   </xacro:macro>

File: robotiq_3f_description/urdf/inc/robotiq_common.xacro (robot description, xacro)
@@ -24,4 +24,5 @@
     <!-- Extract subsections from yaml dictionaries -->
     <xacro:property name="sec_limits" value="${config_joint_limit_parameters['joint_limits']}"/>
+    <xacro:property name="sec_offsets" value="${config_physical_parameters['offsets']}"/>
     <xacro:property name="sec_inertia_parameters" value="${config_physical_parameters['inertia_parameters']}" />
     <xacro:property name="sec_mesh_files" value="${config_visual_parameters['mesh_files']}" />
@@ -122,4 +123,25 @@
     <xacro:property name="finger_link_3_visual_material_color" value="${finger_link_3_mesh['visual']['material']['color']}" scope="parent"/>
     <xacro:property name="finger_link_3_collision_mesh" value="${finger_link_3_mesh['collision']['mesh']}" scope="parent"/>
+    <!-- Origin/Offset parameters -->
+    <xacro:property name="palm_finger_1_joint_origin_xyz" value="${sec_offsets['palm_finger_1_joint']['origin']['xyz']}" scope="parent"/>
+    <xacro:property name="palm_finger_1_joint_origin_rpy" value="${sec_offsets['palm_finger_1_joint']['origin']['rpy']}" scope="parent"/>
+    <xacro:property name="palm_finger_2_joint_origin_xyz" value="${sec_offsets['palm_finger_2_joint']['origin']['xyz']}" scope="parent"/>
+    <xacro:property name="palm_finger_2_joint_origin_rpy" value="${sec_offsets['palm_finger_2_joint']['origin']['rpy']}" scope="parent"/>
+    <xacro:property name="palm_finger_middle_joint_origin_xyz" value="${sec_offsets['palm_finger_middle_joint']['origin']['xyz']}" scope="parent"/>
+    <xacro:property name="palm_finger_middle_joint_origin_rpy" value="${sec_offsets['palm_finger_middle_joint']['origin']['rpy']}" scope="parent"/>
+    <xacro:property name="link_0_origin_xyz" value="${sec_offsets['link_0']['origin']['xyz']}" scope="parent"/>
+    <xacro:property name="link_0_origin_rpy" value="${sec_offsets['link_0']['origin']['rpy']}" scope="parent"/>
+    <xacro:property name="link_1_origin_xyz" value="${sec_offsets['link_1']['origin']['xyz']}" scope="parent"/>
+    <xacro:property name="link_1_origin_rpy" value="${sec_offsets['link_1']['origin']['rpy']}" scope="parent"/>
+    <xacro:property name="link_2_origin_xyz" value="${sec_offsets['link_2']['origin']['xyz']}" scope="parent"/>
+    <xacro:property name="link_2_origin_rpy" value="${sec_offsets['link_2']['origin']['rpy']}" scope="parent"/>
+    <xacro:property name="link_3_origin_xyz" value="${sec_offsets['link_3']['origin']['xyz']}" scope="parent"/>
+    <xacro:property name="link_3_origin_rpy" value="${sec_offsets['link_3']['origin']['rpy']}" scope="parent"/>
+    <xacro:property name="joint_1_origin_xyz" value="${sec_offsets['joint_1']['origin']['xyz']}" scope="parent"/>
+    <xacro:property name="joint_1_origin_rpy" value="${sec_offsets['joint_1']['origin']['rpy']}" scope="parent"/>
+    <xacro:property name="joint_2_origin_xyz" value="${sec_offsets['joint_2']['origin']['xyz']}" scope="parent"/>
+    <xacro:property name="joint_2_origin_rpy" value="${sec_offsets['joint_2']['origin']['rpy']}" scope="parent"/>
+    <xacro:property name="joint_3_origin_xyz" value="${sec_offsets['joint_3']['origin']['xyz']}" scope="parent"/>
+    <xacro:property name="joint_3_origin_rpy" value="${sec_offsets['joint_3']['origin']['rpy']}" scope="parent"/>
   </xacro:macro>
 </robot>
