Commit message: typo fixes

File: robotiq_2f_description/urdf/inc/robotiq_common.xacro (robot description, xacro)
@@ -124,8 +124,8 @@
     <xacro:property name="fingertip_collision_mesh" value="${fingertip_mesh['collision']['mesh']}" scope="parent"/>
     <xacro:property name="finger_pad_mesh" value="${sec_mesh_files['finger_pad']}"/>
-    <xacro:property name="finger_pad_visual_mesh" value="${finger_pad_mesh['visual']['mesh']}" scope="parent"/>
+    <xacro:property name="finger_pad_visual_box_size" value="${finger_pad_mesh['visual']['box_size']}" scope="parent"/>
     <xacro:property name="finger_pad_visual_material_name" value="${finger_pad_mesh['visual']['material']['name']}" scope="parent"/>
     <xacro:property name="finger_pad_visual_material_color" value="${finger_pad_mesh['visual']['material']['color']}" scope="parent"/>
-    <xacro:property name="finger_pad_collision_mesh" value="${finger_pad_mesh['collision']['mesh']}" scope="parent"/>
+    <xacro:property name="finger_pad_collision_box_size" value="${finger_pad_mesh['collision']['box_size']}" scope="parent"/>
   </xacro:macro>
 </robot>

File: robotiq_3f_description/urdf/inc/robotiq_common.xacro (robot description, xacro)
@@ -24,5 +24,4 @@
     <!-- Extract subsections from yaml dictionaries -->
     <xacro:property name="sec_limits" value="${config_joint_limit_parameters['joint_limits']}"/>
-    <!--<xacro:property name="sec_dh_parameters" value="${config_physical_parameters['dh_parameters']}"/>-->
     <xacro:property name="sec_inertia_parameters" value="${config_physical_parameters['inertia_parameters']}" />
     <xacro:property name="sec_mesh_files" value="${config_visual_parameters['mesh_files']}" />
