Commit message: change name of driven joint
-back from 'finger_0_palm_bar' to 'finger_joint'

File: robotiq_2f_description/urdf/inc/finger_macro.xacro (robot description, xacro)
@@ -168,5 +168,5 @@
              effort="${bar_fingertip_joint_effort_limit}"
              velocity="${bar_fingertip_joint_velocity_limit}"/>
-      <mimic joint="finger_0_palm_bar" multiplier="-1" offset="0"/>
+      <mimic joint="finger_joint" multiplier="-1" offset="0"/>
     </joint>
     <joint name="${prefix}fingertip_pad" type="fixed">

File: robotiq_2f_description/urdf/inc/palm_macro.xacro (robot description, xacro)
@@ -34,24 +34,24 @@
     </link>
     <!-- todo: move origin parameters to config files -->
-    <joint name="${prefix}finger_0_palm_bar" type="revolute">
+    <joint name="${prefix}finger_joint" type="revolute">
       <origin xyz="0.0 -0.0306011 0.054904" rpy="0.0 0.0 ${pi}"/>
       <parent link="${prefix}palm"/>
       <child link="${prefix}finger_0_bar_link_0"/>
       <axis xyz="1 0 0"/>
-      <limit lower="${palm_bar_joint_lower_limit}"
-             upper="${palm_bar_joint_upper_limit}"
-             effort="${palm_bar_joint_effort_limit}"
-             velocity="${palm_bar_joint_velocity_limit}"/>
+      <limit lower="${finger_joint_lower_limit}"
+             upper="${finger_joint_upper_limit}"
+             effort="${finger_joint_effort_limit}"
+             velocity="${finger_joint_velocity_limit}"/>
     </joint>
-    <joint name="${prefix}finger_1_palm_bar_mimic" type="revolute">
+    <joint name="${prefix}finger_joint_mimic" type="revolute">
       <origin xyz="0.0 0.0306011 0.054904" rpy="0.0 0.0 0.0"/>
       <parent link="${prefix}palm"/>
       <child link="${prefix}finger_1_bar_link_0"/>
       <axis xyz="1 0 0"/>
-      <limit lower="${palm_bar_joint_lower_limit}"
-             upper="${palm_bar_joint_upper_limit}"
-             effort="${palm_bar_joint_effort_limit}"
-             velocity="${palm_bar_joint_velocity_limit}"/>
-      <mimic joint="${prefix}finger_0_palm_bar" multiplier="1" offset="0" />
+      <limit lower="${finger_joint_lower_limit}"
+             upper="${finger_joint_upper_limit}"
+             effort="${finger_joint_effort_limit}"
+             velocity="${finger_joint_velocity_limit}"/>
+      <mimic joint="${prefix}finger_joint" multiplier="1" offset="0" />
     </joint>
     <joint name="${prefix}finger_0_palm_proximal_phalanx" type="revolute">
@@ -64,5 +64,5 @@
              effort="${palm_proximal_phalanx_joint_effort_limit}"
              velocity="${palm_proximal_phalanx_joint_velocity_limit}"/>
-      <mimic joint="${prefix}finger_0_palm_bar" multiplier="1" offset="0" />
+      <mimic joint="${prefix}finger_joint" multiplier="1" offset="0" />
     </joint>
     <joint name="${prefix}finger_1_palm_proximal_phalanx" type="revolute">
@@ -75,5 +75,5 @@
              effort="${palm_proximal_phalanx_joint_effort_limit}"
              velocity="${palm_proximal_phalanx_joint_velocity_limit}"/>
-      <mimic joint="${prefix}finger_0_palm_bar" multiplier="1" offset="0" />
+      <mimic joint="${prefix}finger_joint" multiplier="1" offset="0" />
     </joint>
   </xacro:macro>

File: robotiq_2f_description/urdf/inc/robotiq_common.xacro (robot description, xacro)
@@ -85,8 +85,8 @@
     <xacro:property name="finger_pad_izz" value="${sec_inertia_parameters['finger_pad']['inertia']['izz']}" scope="parent"/>
     <!-- Joint limit parameters -->
-    <xacro:property name="palm_bar_joint_lower_limit" value="${sec_limits['palm_bar']['min_position']}" scope="parent"/>
-    <xacro:property name="palm_bar_joint_upper_limit" value="${sec_limits['palm_bar']['max_position']}" scope="parent"/>
-    <xacro:property name="palm_bar_joint_velocity_limit" value="${sec_limits['palm_bar']['max_velocity']}" scope="parent"/>
-    <xacro:property name="palm_bar_joint_effort_limit" value="${sec_limits['palm_bar']['max_effort']}" scope="parent"/>
+    <xacro:property name="finger_joint_lower_limit" value="${sec_limits['finger_joint']['min_position']}" scope="parent"/>
+    <xacro:property name="finger_joint_upper_limit" value="${sec_limits['finger_joint']['max_position']}" scope="parent"/>
+    <xacro:property name="finger_joint_velocity_limit" value="${sec_limits['finger_joint']['max_velocity']}" scope="parent"/>
+    <xacro:property name="finger_joint_effort_limit" value="${sec_limits['finger_joint']['max_effort']}" scope="parent"/>
     <xacro:property name="palm_proximal_phalanx_joint_lower_limit" value="${sec_limits['palm_proximal_phalanx']['min_position']}" scope="parent"/>
     <xacro:property name="palm_proximal_phalanx_joint_upper_limit" value="${sec_limits['palm_proximal_phalanx']['max_position']}" scope="parent"/>

File: robotiq_2f_description/urdf/robotiq_2f_macro.xacro (robot description, xacro)
@@ -30,5 +30,5 @@
     />
     <xacro:transmission
-      joint_name="${prefix}finger_0_palm_bar"
+      joint_name="${prefix}finger_joint"
       hw_interface="${transmission_hw_interface}"
     />

File: robotiq_gazebo/urdf/inc/robotiq_2f85_macro.xacro (robot description, xacro)
@@ -20,25 +20,25 @@
       <!-- Configure mimic_joint_plugin for non-driven joints. -->
       <plugin filename="libroboticsgroup_gazebo_mimic_joint_plugin.so" name="${prefix}mimic_0">
-        <joint>${prefix}finger_0_palm_bar</joint>
-        <mimicJoint>${prefix}finger_1_palm_bar_mimic</mimicJoint>
+        <joint>${prefix}finger_joint</joint>
+        <mimicJoint>${prefix}finger_joint_mimic</mimicJoint>
         <multiplier>1.0</multiplier>
       </plugin>
       <plugin filename="libroboticsgroup_gazebo_mimic_joint_plugin.so" name="${prefix}mimic_1">
-        <joint>${prefix}finger_0_palm_bar</joint>
+        <joint>${prefix}finger_joint</joint>
         <mimicJoint>${prefix}finger_0_palm_proximal_phalanx</mimicJoint>
         <multiplier>1.0</multiplier>
       </plugin>
       <plugin filename="libroboticsgroup_gazebo_mimic_joint_plugin.so" name="${prefix}mimic_2">
-        <joint>${prefix}finger_0_palm_bar</joint>
+        <joint>${prefix}finger_joint</joint>
         <mimicJoint>${prefix}finger_1_palm_proximal_phalanx</mimicJoint>
         <multiplier>1.0</multiplier>
       </plugin>
         <plugin filename="libroboticsgroup_gazebo_mimic_joint_plugin.so" name="${prefix}mimic_3">
-        <joint>${prefix}finger_0_palm_bar</joint>
+        <joint>${prefix}finger_joint</joint>
         <mimicJoint>${prefix}finger_1_bar_fingertip</mimicJoint>
         <multiplier>-1.0</multiplier>
       </plugin>
       <plugin filename="libroboticsgroup_gazebo_mimic_joint_plugin.so" name="${prefix}mimic_4">
-        <joint>${prefix}finger_0_palm_bar</joint>
+        <joint>${prefix}finger_joint</joint>
         <mimicJoint>${prefix}finger_0_bar_fingertip</mimicJoint>
         <multiplier>-1.0</multiplier>

Commit message: add origin/offset parameters

File: robotiq_2f_description/urdf/inc/finger_macro.xacro (robot description, xacro)
@@ -153,12 +153,11 @@
       </inertial>
     </link>
-    <!-- todo: move origin parameters to config files -->
     <joint name="${prefix}bar_joint" type="fixed">
-      <origin xyz="0.0 0.0315 -0.0041" rpy="0.0 0.0 0.0"/>
+      <origin xyz="${bar_joint_origin}" rpy="0.0 0.0 0.0"/>
       <parent link="${prefix}bar_link_0"/>
       <child link="${prefix}bar_link_1"/>
     </joint>
     <joint name="${prefix}bar_fingertip" type="revolute">
-      <origin xyz="0.0 0.0061 0.0471" rpy="0.0 0.0 0.0"/>
+      <origin xyz="${bar_fingertip_origin}" rpy="0.0 0.0 0.0"/>
       <parent link="${prefix}bar_link_1"/>
       <child link="${prefix}fingertip"/>
@@ -171,5 +170,5 @@
     </joint>
     <joint name="${prefix}fingertip_pad" type="fixed">
-      <origin xyz="0 -0.0220203446692936 0.03242" rpy="0 0 0"/>
+      <origin xyz="${fingertip_pad_origin}" rpy="0.0 0.0 0.0"/>
       <parent link="${prefix}fingertip"/>
       <child link="${prefix}finger_pad"/>

File: robotiq_2f_description/urdf/inc/palm_macro.xacro (robot description, xacro)
@@ -33,7 +33,6 @@
       </inertial>
     </link>
-    <!-- todo: move origin parameters to config files -->
     <joint name="${prefix}finger_0_palm_bar" type="revolute">
-      <origin xyz="0.0 -0.0306011 0.054904" rpy="0.0 0.0 ${pi}"/>
+      <origin xyz="${finger_joint_origin}" rpy="0.0 0.0 ${pi}"/>
       <parent link="${prefix}palm"/>
       <child link="${prefix}finger_0_bar_link_0"/>
@@ -45,5 +44,5 @@
     </joint>
     <joint name="${prefix}finger_1_palm_bar_mimic" type="revolute">
-      <origin xyz="0.0 0.0306011 0.054904" rpy="0.0 0.0 0.0"/>
+      <origin xyz="${finger_joint_mimic_origin}" rpy="0.0 0.0 0.0"/>
       <parent link="${prefix}palm"/>
       <child link="${prefix}finger_1_bar_link_0"/>
@@ -56,5 +55,5 @@
     </joint>
     <joint name="${prefix}finger_0_palm_proximal_phalanx" type="revolute">
-      <origin xyz="0.0 -0.0127 0.06142" rpy="0.0 0.0 ${pi}"/>
+      <origin xyz="${finger_0_palm_proximal_phalanx_origin}" rpy="0.0 0.0 ${pi}"/>
       <parent link="palm"/>
       <child link="${prefix}finger_0_proximal_phalanx"/>
@@ -67,5 +66,5 @@
     </joint>
     <joint name="${prefix}finger_1_palm_proximal_phalanx" type="revolute">
-      <origin xyz="0.0 0.0127 0.06142" rpy="0.0 0.0 0.0"/>
+      <origin xyz="${finger_1_palm_proximal_phalanx_origin}" rpy="0.0 0.0 0.0"/>
       <parent link="palm"/>
       <child link="${prefix}finger_1_proximal_phalanx"/>

File: robotiq_2f_description/urdf/inc/robotiq_common.xacro (robot description, xacro)
@@ -24,4 +24,5 @@
     <!-- Extract subsections from yaml dictionaries -->
     <xacro:property name="sec_limits" value="${config_joint_limit_parameters['joint_limits']}"/>
+    <xacro:property name="sec_offsets" value="${config_physical_parameters['offsets']}"/>
     <xacro:property name="sec_inertia_parameters" value="${config_physical_parameters['inertia_parameters']}" />
     <xacro:property name="sec_mesh_files" value="${config_visual_parameters['mesh_files']}" />
@@ -128,4 +129,12 @@
     <xacro:property name="finger_pad_visual_material_color" value="${finger_pad_mesh['visual']['material']['color']}" scope="parent"/>
     <xacro:property name="finger_pad_collision_box_size" value="${finger_pad_mesh['collision']['box_size']}" scope="parent"/>
+    <!-- Origin/Offset parameters -->
+    <xacro:property name="finger_joint_origin" value="${sec_offsets['finger_joint']['origin']['xyz']}" scope="parent"/>
+    <xacro:property name="finger_joint_mimic_origin" value="${sec_offsets['finger_joint_mimic']['origin']['xyz']}" scope="parent"/>
+    <xacro:property name="finger_0_palm_proximal_phalanx_origin" value="${sec_offsets['finger_0_palm_proximal_phalanx']['origin']['xyz']}" scope="parent"/>
+    <xacro:property name="finger_1_palm_proximal_phalanx_origin" value="${sec_offsets['finger_1_palm_proximal_phalanx']['origin']['xyz']}" scope="parent"/>
+    <xacro:property name="bar_joint_origin" value="${sec_offsets['bar_joint']['origin']['xyz']}" scope="parent"/>
+    <xacro:property name="bar_fingertip_origin" value="${sec_offsets['bar_fingertip']['origin']['xyz']}" scope="parent"/>
+    <xacro:property name="fingertip_pad_origin" value="${sec_offsets['fingertip_pad']['origin']['xyz']}" scope="parent"/>
   </xacro:macro>
 </robot>

Commit message: change (driven) joint name back to origin name
-change from 'finger_0_palm_bar' to 'finger_joint'

File: robotiq_2f_description/urdf/inc/finger_macro.xacro (robot description, xacro)
@@ -167,5 +167,5 @@
              effort="${bar_fingertip_joint_effort_limit}"
              velocity="${bar_fingertip_joint_velocity_limit}"/>
-      <mimic joint="finger_0_palm_bar" multiplier="-1" offset="0"/>
+      <mimic joint="finger_joint" multiplier="-1" offset="0"/>
     </joint>
     <joint name="${prefix}fingertip_pad" type="fixed">

File: robotiq_2f_description/urdf/inc/palm_macro.xacro (robot description, xacro)
@@ -33,24 +33,24 @@
       </inertial>
     </link>
-    <joint name="${prefix}finger_0_palm_bar" type="revolute">
+    <joint name="${prefix}finger_joint" type="revolute">
       <origin xyz="${finger_joint_origin}" rpy="0.0 0.0 ${pi}"/>
       <parent link="${prefix}palm"/>
       <child link="${prefix}finger_0_bar_link_0"/>
       <axis xyz="1 0 0"/>
-      <limit lower="${palm_bar_joint_lower_limit}"
-             upper="${palm_bar_joint_upper_limit}"
-             effort="${palm_bar_joint_effort_limit}"
-             velocity="${palm_bar_joint_velocity_limit}"/>
+      <limit lower="${finger_joint_lower_limit}"
+             upper="${finger_joint_upper_limit}"
+             effort="${finger_joint_effort_limit}"
+             velocity="${finger_joint_velocity_limit}"/>
     </joint>
-    <joint name="${prefix}finger_1_palm_bar_mimic" type="revolute">
+    <joint name="${prefix}finger_joint_mimic" type="revolute">
       <origin xyz="${finger_joint_mimic_origin}" rpy="0.0 0.0 0.0"/>
       <parent link="${prefix}palm"/>
       <child link="${prefix}finger_1_bar_link_0"/>
       <axis xyz="1 0 0"/>
-      <limit lower="${palm_bar_joint_lower_limit}"
-             upper="${palm_bar_joint_upper_limit}"
-             effort="${palm_bar_joint_effort_limit}"
-             velocity="${palm_bar_joint_velocity_limit}"/>
-      <mimic joint="${prefix}finger_0_palm_bar" multiplier="1" offset="0" />
+      <limit lower="${finger_joint_lower_limit}"
+             upper="${finger_joint_upper_limit}"
+             effort="${finger_joint_effort_limit}"
+             velocity="${finger_joint_velocity_limit}"/>
+      <mimic joint="${prefix}finger_joint" multiplier="1" offset="0" />
     </joint>
     <joint name="${prefix}finger_0_palm_proximal_phalanx" type="revolute">
@@ -63,5 +63,5 @@
              effort="${palm_proximal_phalanx_joint_effort_limit}"
              velocity="${palm_proximal_phalanx_joint_velocity_limit}"/>
-      <mimic joint="${prefix}finger_0_palm_bar" multiplier="1" offset="0" />
+      <mimic joint="${prefix}finger_joint" multiplier="1" offset="0" />
     </joint>
     <joint name="${prefix}finger_1_palm_proximal_phalanx" type="revolute">
@@ -74,5 +74,5 @@
              effort="${palm_proximal_phalanx_joint_effort_limit}"
              velocity="${palm_proximal_phalanx_joint_velocity_limit}"/>
-      <mimic joint="${prefix}finger_0_palm_bar" multiplier="1" offset="0" />
+      <mimic joint="${prefix}finger_joint" multiplier="1" offset="0" />
     </joint>
   </xacro:macro>

File: robotiq_2f_description/urdf/inc/robotiq_common.xacro (robot description, xacro)
@@ -86,8 +86,8 @@
     <xacro:property name="finger_pad_izz" value="${sec_inertia_parameters['finger_pad']['inertia']['izz']}" scope="parent"/>
     <!-- Joint limit parameters -->
-    <xacro:property name="palm_bar_joint_lower_limit" value="${sec_limits['palm_bar']['min_position']}" scope="parent"/>
-    <xacro:property name="palm_bar_joint_upper_limit" value="${sec_limits['palm_bar']['max_position']}" scope="parent"/>
-    <xacro:property name="palm_bar_joint_velocity_limit" value="${sec_limits['palm_bar']['max_velocity']}" scope="parent"/>
-    <xacro:property name="palm_bar_joint_effort_limit" value="${sec_limits['palm_bar']['max_effort']}" scope="parent"/>
+    <xacro:property name="finger_joint_lower_limit" value="${sec_limits['finger_joint']['min_position']}" scope="parent"/>
+    <xacro:property name="finger_joint_upper_limit" value="${sec_limits['finger_joint']['max_position']}" scope="parent"/>
+    <xacro:property name="finger_joint_velocity_limit" value="${sec_limits['finger_joint']['max_velocity']}" scope="parent"/>
+    <xacro:property name="finger_joint_effort_limit" value="${sec_limits['finger_joint']['max_effort']}" scope="parent"/>
     <xacro:property name="palm_proximal_phalanx_joint_lower_limit" value="${sec_limits['palm_proximal_phalanx']['min_position']}" scope="parent"/>
     <xacro:property name="palm_proximal_phalanx_joint_upper_limit" value="${sec_limits['palm_proximal_phalanx']['max_position']}" scope="parent"/>
